File: PROJET KICAD/Robot2025LabyrintheTemplate.kicad_sch (KiCad schematic)
At the start: 23 parts, among them J1 HC-SR04 gauche, J10 CAPTEUR TOF _BAS, J11 SERVO MOTEUR 4, J2 +VBatt, J3 SERVO MOTEUR 1, J4 SERVO MOTEUR 2, J5 cap sen0101, J7 SERVO MOTEUR 3, J8 HC-SR04 droite, J9 CAPTEUR TOF_HAUT, U1 module_mpu6050, U3 NRF24L01P-Module-E01ML01DP5_B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

Commit message: revue avec alaime
Parts:
- removed C1, C2: 10uF, ISI-Capacitor:WCAP-ATUL_18X35.5_DXL_, symbol ISI-Capacitor:860040781020
- removed J10: CAPTEUR TOF _BAS, ISI-Connector_PinHeader_2.54mm:PinHeader_1x06_P2.54mm_Long_Vertical, symbol ISI-Connector_PinHeader_2.54mm:Conn_01x06_Pin
- removed J2: +VBatt, ISI-Connector_JST:JST_XH_B2B-XH-AM_1x02_P2.50mm_Long_Vertical, symbol ISI-Connector_JST:Conn_01x02_Pin
- removed J9: CAPTEUR TOF_HAUT, ISI-Connector_PinHeader_2.54mm:PinHeader_1x06_P2.54mm_Long_Vertical, symbol ISI-Connector_PinHeader_2.54mm:Conn_01x06_Pin
- removed U3: NRF24L01P-Module-E01ML01DP5_Breakout, ISI-Modules:E01-ML01DP5, symbol ISI-Modules:NRF24L01P-Module-E01ML01DP5_Breakout
- added C1, C2: C_Gen, ISI-Capacitor:C_1206_3216Metric_Pad1.33x1.80mm_HandSolder, symbol ISI-Capacitor:C_1206
- added C4: C_Polarized, ISI-Capacitor:CP_EIA-6032-28_Kemet-C_Pad2.25x2.35mm_HandSolder, symbol ISI-Capacitor:C_Polarized
- added F1: Fuse, ISI-Divers:Fuseholder_TR5_Littelfuse_No560_No460, symbol ISI-Divers:Fuse
- added J12, J6: Conn_01x06_Pin, ISI-Connector_PinHeader_2.54mm:PinHeader_1x06_P2.54mm_Long_Vertical, symbol ISI-Connector_PinHeader_2.54mm:Conn_01x06_Pin
- added J13, J16: Conn_01x05_Pin, ISI-Connector_JST:JST_XH_B5B-XH-AM_1x05_P2.50mm_Long_Vertical, symbol ISI-Connector_JST:Conn_01x05_Pin
- added J14, J18: Conn_01x02_Pin, ISI-Connector_JST:JST_XH_B2B-XH-AM_1x02_P2.50mm_Long_Vertical, symbol ISI-Connector_JST:Conn_01x02_Pin
- added J15: CON 1x2 POLARIZED, ISI-Connector_Generic:AMASS_XT60-F_1x02_P7.20mm_Vertical, symbol ISI-Connector_Generic:XT60_F
- added J17, J19: Conn_01x04_Pin, ISI-Connector_JST:JST_XH_B4B-XH-AM_1x04_P2.50mm_Long_Vertical, symbol ISI-Connector_JST:Conn_01x04_Pin
- added R2, R3: 10k, ISI-Resistor:R_1206_3216Metric_Pad1.30x1.75mm_HandSolder, symbol ISI-Resistor:R_US_1206
- added U2: LM1117MPX-3.3, ISI-IC:SOT-223-3_TabPin2, symbol ISI-IC:LM1117MPX-3.3
- added U4: NRF24L01P-Module-E01ML01DP5_Breakout, ISI-Modules:E01-ML01DP5, symbol ISI-Modules:NRF24L01P-Module-E01ML01DP5_Breakout
Connections:
- net T_SCL is gone; now on an unnamed net: A2.D21 (D21/SCL)
- net T_SDA is gone; now on an unnamed net: A2.D20 (D20/SDA)
- net +5V: now also J3.2 (Pin_2), C2.1, J13.1 (Pin_1), J16.1 (Pin_1), J18.1 (Pin_1), R2.1, R3.1, U2.3 (VI); no longer A1.10 (M0), A1.11 (M1), A1.12 (M2)
- net D_CE: now also U4.3 (CE)
- net D_CSN: now also U4.4 (~{CSN})
- net D_MISO: now also U4.7 (MISO)
- net D_MOSI: now also U4.6 (MOSI)
- net D_SCK: now also U4.5 (SCK)
- net D_XSHUT_B: now also J13.5 (Pin_5)
- net D_XSHUT_H: now also J16.5 (Pin_5)
- net GND: now also A1.10 (M0), A1.11 (M1), A1.12 (M2), A5.7 (GND), C1.2, C2.2, C4.2, J13.2 (Pin_2), J14.2 (Pin_2), J15.2, J16.2 (Pin_2), J18.2 (Pin_2), U2.1 (GND), U4.1 (GND)
- net Vin: now also A5.8 (VMOT), J14.1 (Pin_1); no longer A2.VIN
- net at D3.2 (A): now also F1.2
- net at A5.3 (A2): now also A5.4 (A1), J17.1 (Pin_1)
- net at A5.5 (B1): now also J17.3 (Pin_3)
- net at A5.6 (B2): now also J17.4 (Pin_4)
- net at A1.3 (A2): now also J12.3 (Pin_3)
- net at A1.4 (A1): now also J12.2 (Pin_2)
- net at A1.5 (B1): now also J12.4 (Pin_4)
- net at A1.6 (B2): now also J12.5 (Pin_5)
- net at A1.7 (GND): now also J12.6 (Pin_6)
- net at A1.8 (VMOT): now also J12.1 (Pin_1)
- net at A3.3 (A2): now also J6.3 (Pin_3)
- net at A3.4 (A1): now also J6.2 (Pin_2)
- net at A3.5 (B1): now also J6.4 (Pin_4)
- net at A3.6 (B2): now also J6.5 (Pin_5)
- net at A3.7 (GND): now also J6.6 (Pin_6)
- net at A3.8 (VMOT): now also J6.1 (Pin_1)
- net at A4.3 (A2): now also J19.3 (Pin_3)
- net at A4.4 (A1): now also J19.4 (Pin_4)
- net +3V3: no longer names the net of A2.3V3 (3.3V)
- net SCL_1: no longer names the net of U1.3 (SCL)
- net SCL_1: now also J13.3 (Pin_3), J16.3 (Pin_3), R3.2; no longer A2.SCL
- net SDA_1: no longer names the net of U1.4 (SDA)
- net SDA_1: now also J13.4 (Pin_4), J16.4 (Pin_4), R2.2; no longer A2.SDA
- new net: F1.1, J15.1
- new net: C1.1, C4.1, U2.2 (VO), U4.2 (VCC)
- new net: J19.1 (Pin_1), J19.2 (Pin_2)
- no-connect marks 82 -> 59
Other:
- note added: "A1"
- note added: "A2"
- note added: "B1"
- note added: "B2"
- note added: "GND"
- note added: "SCL SDA"
- note added: "VIN"
- note removed: "Exemple connecteur JST."
- moved on the sheet: A1, A3, A4, A5, J11, J3, J4, J5, J7, J8, U1
