File: PROJET KICAD/Robot2025LabyrintheTemplate.kicad_sch (KiCad schematic)
At the start: 34 parts, among them J1 HC-SR04 gauche, J11 SERVO MOTEUR 4, J12 Conn_01x06_Pin, J13 Conn_01x05_Pin, J14 Conn_01x02_Pin, J15 CON 1x2 POLARIZED, J16 Conn_01x05_Pin, J17 Conn_01x04_Pin, J18 Conn_01x02_Pin, J19 Conn_01x04_Pin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

Commit message: test2
Other:
- moved on the sheet: J5
Changed lines of the file:
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@@
 	(wire
 		(pts
-			(xy 261.62 74.93) (xy 264.16 74.93)
+			(xy 323.85 82.55) (xy 326.39 82.55)
 		)
 		(stroke
@@
 	(wire
 		(pts
-			(xy 241.3 77.47) (xy 248.92 77.47)
+			(xy 303.53 85.09) (xy 311.15 85.09)
 		)
 		(stroke
@@
 	(wire
 		(pts
-			(xy 261.62 69.85) (xy 266.7 69.85)
+			(xy 323.85 77.47) (xy 328.93 77.47)
 		)
 		(stroke
@@
 	(wire
 		(pts
-			(xy 241.3 74.93) (xy 248.92 74.93)
+			(xy 303.53 82.55) (xy 311.15 82.55)
 		)
 		(stroke
@@
 	(wire
 		(pts
-			(xy 261.62 72.39) (xy 265.43 72.39)
+			(xy 323.85 80.01) (xy 327.66 80.01)
 		)
 		(stroke
@@
 	(wire
 		(pts
-			(xy 261.62 77.47) (xy 265.43 77.47)
+			(xy 323.85 85.09) (xy 327.66 85.09)
 		)
 		(stroke
@@
 	(wire
 		(pts
-			(xy 242.57 72.39) (xy 248.92 72.39)
+			(xy 304.8 80.01) (xy 311.15 80.01)
 		)
 		(stroke
@@
 	(wire
 		(pts
-			(xy 240.03 68.58) (xy 240.03 69.85)
+			(xy 302.26 76.2) (xy 302.26 77.47)
 		)
 		(stroke
@@
 	(wire
 		(pts
-			(xy 240.03 69.85) (xy 248.92 69.85)
+			(xy 302.26 77.47) (xy 311.15 77.47)
 		)
 		(stroke
@@
 	)
 	(label "GND"
-		(at 247.65 77.47 270)
+		(at 309.88 85.09 270)
 		(effects
 			(font
@@
 	)
 	(label "D_S0"
-		(at 266.7 69.85 0)
+		(at 328.93 77.47 0)
 		(effects
 			(font
@@
 	)
 	(label "D_OUT"
-		(at 242.57 72.39 0)
+		(at 304.8 80.01 0)
 		(effects
 			(font
@@
 	)
 	(label "D_S2"
-		(at 264.16 74.93 0)
+		(at 326.39 82.55 0)
 		(effects
 			(font
@@
 	)
 	(label "D_S3"
-		(at 265.43 77.47 0)
+		(at 327.66 85.09 0)
 		(effects
 			(font
@@
 	)
 	(label "D_S1"
-		(at 265.43 72.39 0)
+		(at 327.66 80.01 0)
 		(effects
 			(font
@@
 	(symbol
 		(lib_id "power:GND")
-		(at 240.03 68.58 180)
+		(at 302.26 76.2 180)
 		(unit 1)
 		(body_style 1)
@@
 		(dnp no)
 		(property "Reference" "#PWR019"
-			(at 240.03 62.23 0)
+			(at 302.26 69.85 0)
 			(hide yes)
 			(show_name no)
@@
 		)
 		(property "Value" "GND"
-			(at 240.03 63.5 0)
+			(at 302.26 71.12 0)
 			(show_name no)
 			(do_not_autoplace no)
@@
 		)
 		(property "Footprint" ""
-			(at 240.03 68.58 0)
+			(at 302.26 76.2 0)
 			(hide yes)
 			(show_name no)
@@
 		)
 		(property "Datasheet" ""
-			(at 240.03 68.58 0)
+			(at 302.26 76.2 0)
 			(hide yes)
 			(show_name no)
@@
 		)
 		(property "Description" "Power symbol creates a global label with name \"GND\" , ground"
-			(at 240.03 68.58 0)
+			(at 302.26 76.2 0)
 			(hide yes)
 			(show_name no)
@@
 	(symbol
 		(lib_id "ISI-Connector_PinSocket_2.54mm:Conn_02x04_Odd_Even")
-		(at 254 72.39 0)
+		(at 316.23 80.01 0)
 		(unit 1)
 		(body_style 1)
@@
 		(dnp no)
 		(property "Reference" "J5"
-			(at 255.27 63.5 0)
+			(at 317.5 71.12 0)
 			(show_name no)
 			(do_not_autoplace no)
@@
 		)
 		(property "Value" "cap sen0101"
-			(at 255.27 66.04 0)
+			(at 317.5 73.66 0)
 			(show_name no)
 			(do_not_autoplace no)
@@
 		)
 		(property "Footprint" "ISI-Connector_PinSocket_2.54mm:PinSocket_2x04_P2.54mm_Vertical"
-			(at 254 72.39 0)
+			(at 316.23 80.01 0)
 			(hide yes)
 			(show_name no)
@@
 		)
 		(property "Datasheet" ""
-			(at 254 72.39 0)
+			(at 316.23 80.01 0)
 			(hide yes)
 			(show_name no)
@@
 		)
 		(property "Description" "Generic connector, double row, 02x04, odd/even pin numbering scheme (row 1 odd numbers, row 2 even numbers), script generated (kicad-library-utils/schlib/autogen/connector/)"
-			(at 254 72.39 0)
+			(at 316.23 80.01 0)
 			(hide yes)
 			(show_name no)
@@
 	(symbol
 		(lib_id "power:GND")
-		(at 241.3 77.47 270)
+		(at 303.53 85.09 270)
 		(unit 1)
 		(body_style 1)
@@
 		(dnp no)
 		(property "Reference" "#PWR020"
-			(at 234.95 77.47 0)
+			(at 297.18 85.09 0)
 			(hide yes)
 			(show_name no)
@@
 		)
 		(property "Value" "GND"
-			(at 236.22 77.47 90)
+			(at 298.45 85.09 90)
 			(show_name no)
 			(do_not_autoplace no)
@@
 		)
 		(property "Footprint" ""
-			(at 241.3 77.47 0)
+			(at 303.53 85.09 0)
 			(hide yes)
 			(show_name no)
@@
 		)
 		(property "Datasheet" ""
-			(at 241.3 77.47 0)
+			(at 303.53 85.09 0)
 			(hide yes)
 			(show_name no)
@@
 		)
 		(property "Description" "Power symbol creates a global label with name \"GND\" , ground"
-			(at 241.3 77.47 0)
+			(at 303.53 85.09 0)
 			(hide yes)
 			(show_name no)
@@
 	(symbol
 		(lib_id "power:+5V")
-		(at 241.3 74.93 90)
+		(at 303.53 82.55 90)
 		(unit 1)
 		(body_style 1)
@@
 		(fields_autoplaced yes)
 		(property "Reference" "#PWR021"
-			(at 245.11 74.93 0)
+			(at 307.34 82.55 0)
 			(hide yes)
 			(show_name no)
@@
 		)
 		(property "Value" "+5V"
-			(at 237.49 74.9299 90)
+			(at 299.72 82.5499 90)
 			(show_name no)
 			(do_not_autoplace no)
@@
 		)
 		(property "Footprint" ""
-			(at 241.3 74.93 0)
+			(at 303.53 82.55 0)
 			(hide yes)
 			(show_name no)
@@
 		)
 		(property "Datasheet" ""
-			(at 241.3 74.93 0)
+			(at 303.53 82.55 0)
 			(hide yes)
 			(show_name no)
@@
 		)
 		(property "Description" "Power symbol creates a global label with name \"+5V\""
-			(at 241.3 74.93 0)
+			(at 303.53 82.55 0)
 			(hide yes)
 			(show_name no)
