File: PROJET KICAD/Robot2025LabyrintheTemplate.kicad_pcb (KiCad board)
At the start: 2 copper layers, 210 x 85 mm, 35 parts, among them J1 HC-SR04 gauche, J11 SERVO MOTEUR 4, J13 capteur TOF BAS, J14 Vinput regul, J15 CON 1x2 POLARIZED, J16 capteur TOF HAUT, J17 moteur 2 AV, J18 Vout regul, J2 cap sen0101, J20 moteur 3 DR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

Commit message: final
Parts:
- moved J4 1.50 mm to (221.0, 123.5)
- moved J17 1.50 mm to (229.5, 125.0)
- moved D2 1.03 mm to (81.0, 96.5)
Routing:
- net /wht_2: track 242.0 -> 220.3 mm
- net +5V: track 97.1 -> 86.5 mm
- net /Vin: track 288.4 -> 285.9 mm
- net /D_INT: track 27.2 -> 28.1 mm
- net /wht_1: track 90.9 -> 91.4 mm, vias 2 -> 4
- net /D_OUT: vias 0 -> 2
Other:
- board size 210 x 85 mm -> 200 x 85 mm

Commit message: Différentes modifs à discuter de vive voix
Parts:
- added R5: 0R, ISI-Resistor:R_1206_3216Metric_Pad1.30x1.75mm_HandSolder, B.Cu at (185.9, 106.7)
- added R6: 0R, ISI-Resistor:R_1206_3216Metric_Pad1.30x1.75mm_HandSolder, B.Cu at (185.9, 104.1)
- C1, C2, C4, U2: moved to B.Cu
- moved C2 51.9 mm to (213.3, 76.2)
- moved U2 43.7 mm to (214.9, 81.3), turned to 0 degrees
- moved C4 40.2 mm to (208.3, 80.3), turned to 90 degrees
- moved C1 29.3 mm to (214.9, 86.9), turned to 180 degrees
- moved D3 3.50 mm to (68.8, 97.0)
- moved D2 1.81 mm to (82.8, 96.4)
Connections:
- A2 pad D49: /D_CSN -> Net-(A2-PadD49)
- A2 pad D53: unconnected-(A2-D53_CS-PadD53) -> Net-(A2-D53_CS)
- A5 pad 10: +5V -> GND
- A5 pad 11: +5V -> GND
- A5 pad 12: +5V -> GND
Routing:
- net GND: track 68.1 -> 28.1 mm
- net Net-(U2-VO): track 52.6 -> 20.5 mm, vias 2 -> 0
- net /Vin: track 285.9 -> 307.7 mm
- net +5V: track 86.5 -> 95.0 mm, vias 5 -> 7
- net /d2-STEP: track 142.2 -> 149.3 mm
- net Net-(A2-D53_CS): track 0.00 -> 5.63 mm
- net /D_CSN: track 43.1 -> 37.9 mm, vias 2 -> 3
- net /d2-ENABLE: track 121.9 -> 126.9 mm
- net Net-(A2-PadD49): track 0.00 -> 4.58 mm
- net Net-(A5-A1): track 0.54 -> 4.21 mm
- net Net-(A5-A2): track 0.00 -> 2.83 mm
- net Net-(F1-Pad1): track 11.4 -> 12.9 mm
- net Net-(D3-A): track 9.24 -> 7.72 mm
- net Net-(D3-K): track 36.2 -> 37.6 mm, vias 2 -> 1
- net /D_MISO: track 44.8 -> 46.1 mm
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